File: eagle/3dring.brd (EAGLE design)
At the start: 43 x 18 mm, 19 parts, among them CN2 M02JST-PTH-2, IC7 TLV71333DBV, U1 WS2811, U3 ATMEGA328, Y1 8Mhz

Commit message: Updated board problems
Routing:
- net VCC: track 77.5 -> 63.0 mm
Changed lines of the file:
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@@
 <setting verticaltext="up"/>
 </settings>
-<grid distance="0.5" unitdist="mm" unit="mm" style="lines" multiple="1" display="yes" altdistance="0.025" altunitdist="inch" altunit="inch"/>
+<grid distance="0.1" unitdist="mm" unit="mm" style="lines" multiple="1" display="yes" altdistance="0.025" altunitdist="inch" altunit="inch"/>
 <layers>
 <layer number="1" name="Top" color="4" fill="1" visible="yes" active="yes"/>
@@
 <wire x1="32.5" y1="7.6" x2="32.4" y2="7.7" width="0.4064" layer="1"/>
 <wire x1="32.4" y1="7.7" x2="32.4" y2="9.55" width="0.4064" layer="1"/>
-<wire x1="32.4" y1="9.55" x2="31.55" y2="9.55" width="0.4064" layer="1"/>
-<wire x1="31.55" y1="9.55" x2="30.9" y2="10.2" width="0.4064" layer="1"/>
-<wire x1="30.9" y1="10.2" x2="30.9" y2="13.3" width="0.4064" layer="1"/>
-<wire x1="30.9" y1="13.3" x2="32.3" y2="14.7" width="0.4064" layer="1"/>
-<wire x1="32.3" y1="14.7" x2="32.3" y2="16.3" width="0.4064" layer="1"/>
-<wire x1="32.3" y1="16.3" x2="31.5" y2="17.1" width="0.4064" layer="1"/>
-<wire x1="31.5" y1="17.1" x2="26.62" y2="17.1" width="0.4064" layer="1"/>
 <wire x1="19.31816875" y1="11.75248125" x2="17.4656875" y2="9.9" width="0.4064" layer="1"/>
 <wire x1="17.4656875" y1="9.9" x2="15.3" y2="9.9" width="0.4064" layer="1"/>

Commit message: New version
Parts:
- moved JP2 5.10 mm to (30.5, 15.9), turned to 180 degrees
Connections:
- net IRDETECT: now also U3.9; no longer U3.1
- net IRLED: now also U3.1; no longer U3.9
- net RX-I: now also JP3.3; no longer JP3.2
- net TX-O: now also JP3.2; no longer JP3.3
Routing:
- net IRDETECT: track 8.33 -> 20.4 mm
- net IRLED: track 26.5 -> 17.2 mm, vias 1 -> 0
- net IRPWR: track 12.2 -> 8.08 mm, vias 1 -> 0
- net RX-I: track 7.37 -> 9.18 mm
- net TX-O: track 7.98 -> 7.60 mm, vias 0 -> 2
Other:
- board text added: "3DRing V0.2"
- board text removed: "3DRing V0.1"
Changed lines of the file:
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@@
 <hole x="40" y="11.5" drill="2.2"/>
 <text x="26.4" y="13.5" size="0.8128" layer="25">IR rec.</text>
-<text x="31.8" y="6.5" size="0.8128" layer="25" rot="R270">3DeWitt</text>
-<text x="33.1" y="6.5" size="0.8128" layer="25" rot="R270">IdleHands</text>
-<text x="42.5" y="10.9" size="0.8128" layer="25" rot="R90">3DRing V0.1</text>
+<text x="31.8" y="5" size="0.8128" layer="25" font="vector" rot="R270">3DeWitt</text>
+<text x="33" y="6.8" size="0.8128" layer="25" font="vector" rot="R270">IdleHands</text>
+<text x="42.4" y="10" size="0.8128" layer="25" font="vector" rot="R90">3DRing V0.2</text>
 </plain>
 <attributes>
@@
 </autorouter>
 <elements>
-<element name="JP2" library="SparkFun" package="1X03" value="" x="25.4" y="15.9" smashed="yes">
-<attribute name="VALUE" x="24.13" y="12.725" size="1.27" layer="27"/>
+<element name="JP2" library="SparkFun" package="1X03" value="" x="30.5" y="15.9" smashed="yes" rot="R180">
+<attribute name="VALUE" x="31.77" y="19.075" size="1.27" layer="27" rot="R180"/>
 </element>
 <element name="C5" library="SparkFun" package="0402-CAP" value="0.1uF" x="11.1" y="4.02" smashed="yes" rot="R270">
@@
 </element>
 <element name="IR" library="SparkFun-LED" package="LED5MM" value="" x="37" y="16" smashed="yes">
-<attribute name="NAME" x="40.075" y="16.5334" size="0.6096" layer="25" ratio="10"/>
+<attribute name="NAME" x="40.5666" y="14.175" size="0.6096" layer="25" ratio="10" rot="R90"/>
 <attribute name="VALUE" x="40.2004" y="14.1966" size="1.27" layer="27" ratio="10"/>
 </element>
@@
 <via x="29.5" y="12.1" extent="1-16" drill="0.4318"/>
 <via x="27.5" y="10.7" extent="1-16" drill="0.4318"/>
-<via x="22.8" y="6.6" extent="1-16" drill="0.4318"/>
+<via x="22.4" y="6.7" extent="1-16" drill="0.4318"/>
 <via x="22.1" y="4.3" extent="1-16" drill="0.4318"/>
 <via x="33.9" y="12" extent="1-16" drill="0.4318"/>
@@
 <signal name="IRDETECT">
 <contactref element="JP2" pad="1"/>
-<contactref element="U3" pad="1"/>
-<wire x1="21.015225" y1="10.055425" x2="21.6598" y2="10.7" width="0.4064" layer="1"/>
-<wire x1="21.6598" y1="10.7" x2="22.8" y2="10.7" width="0.4064" layer="1"/>
-<wire x1="22.8" y1="10.7" x2="25.4" y2="13.3" width="0.4064" layer="1"/>
-<wire x1="25.4" y1="13.3" x2="25.4" y2="15.9" width="0.4064" layer="1"/>
+<contactref element="U3" pad="9"/>
+<wire x1="30.5" y1="15.9" x2="30.2" y2="15.9" width="0.3048" layer="1"/>
+<wire x1="30.2" y1="15.9" x2="28.9" y2="17.2" width="0.3048" layer="1"/>
+<wire x1="28.9" y1="17.2" x2="14.7" y2="17.2" width="0.3048" layer="1"/>
+<wire x1="14.7" y1="17.2" x2="13.8" y2="16.3" width="0.3048" layer="1"/>
+<wire x1="13.8" y1="16.3" x2="13.8" y2="15.159796875" width="0.3048" layer="1"/>
+<wire x1="13.8" y1="15.159796875" x2="14.944571875" y2="14.015225" width="0.3048" layer="1"/>
 </signal>
 <signal name="RESET">
@@
 <signal name="RX-I">
 <contactref element="U3" pad="30"/>
-<contactref element="JP3" pad="2"/>
 <wire x1="19.883853125" y1="6.8132" x2="21.497053125" y2="5.2" width="0.3" layer="1"/>
-<wire x1="21.497053125" y1="5.2" x2="24.6" y2="5.2" width="0.3" layer="1"/>
-<wire x1="24.6" y1="5.2" x2="25.46" y2="4.34" width="0.3" layer="1"/>
-<wire x1="25.46" y1="4.34" x2="25.46" y2="3.57" width="0.3" layer="1"/>
+<contactref element="JP3" pad="3"/>
+<wire x1="21.497053125" y1="5.2" x2="23.5" y2="5.2" width="0.3048" layer="1"/>
+<wire x1="23.5" y1="5.2" x2="24.3" y2="6" width="0.3048" layer="1"/>
+<wire x1="24.3" y1="6" x2="25" y2="6" width="0.3048" layer="1"/>
+<wire x1="25" y1="6" x2="26.5" y2="4.5" width="0.3048" layer="1"/>
+<wire x1="26.5" y1="4.5" x2="26.5" y2="3.61" width="0.3048" layer="1"/>
+<wire x1="26.5" y1="3.61" x2="26.46" y2="3.57" width="0.3048" layer="1"/>
 </signal>
 <signal name="TX-O">
 <contactref element="U3" pad="31"/>
-<contactref element="JP3" pad="3"/>
 <wire x1="20.4495375" y1="7.378884375" x2="22.028421875" y2="5.8" width="0.3" layer="1"/>
-<wire x1="22.028421875" y1="5.8" x2="24.9" y2="5.8" width="0.3" layer="1"/>
-<wire x1="24.9" y1="5.8" x2="26.46" y2="4.24" width="0.3" layer="1"/>
-<wire x1="26.46" y1="4.24" x2="26.46" y2="3.57" width="0.3" layer="1"/>
+<contactref element="JP3" pad="2"/>
+<wire x1="22.028421875" y1="5.8" x2="22.9" y2="5.8" width="0.3048" layer="1"/>
+<wire x1="22.9" y1="5.8" x2="23.3" y2="6.2" width="0.3048" layer="1"/>
+<via x="23.3" y="6.2" extent="1-16" drill="0.4318"/>
+<wire x1="23.3" y1="6.2" x2="23.7" y2="6.2" width="0.3048" layer="16"/>
+<wire x1="23.7" y1="6.2" x2="24.8" y2="5.1" width="0.3048" layer="16"/>
+<via x="24.8" y="5.1" extent="1-16" drill="0.4318"/>
+<wire x1="24.8" y1="5.1" x2="25.1" y2="5.1" width="0.3048" layer="1"/>
+<wire x1="25.1" y1="5.1" x2="25.4" y2="4.8" width="0.3048" layer="1"/>
+<wire x1="25.4" y1="4.8" x2="25.4" y2="3.63" width="0.3048" layer="1"/>
+<wire x1="25.4" y1="3.63" x2="25.46" y2="3.57" width="0.3048" layer="1"/>
 </signal>
 <signal name="IRPWR">
 <contactref element="U3" pad="2"/>
 <contactref element="JP2" pad="3"/>
-<wire x1="20.4495375" y1="10.6211125" x2="22.228425" y2="12.4" width="0.4064" layer="1"/>
-<wire x1="22.228425" y1="12.4" x2="22.7" y2="12.4" width="0.4064" layer="1"/>
-<via x="22.7" y="12.4" extent="1-16" drill="0.6"/>
-<wire x1="22.7" y1="12.4" x2="26.98" y2="12.4" width="0.4064" layer="16"/>
-<wire x1="26.98" y1="12.4" x2="30.48" y2="15.9" width="0.4064" layer="16"/>
+<wire x1="25.42" y1="15.9" x2="25.42" y2="14.82" width="0.3048" layer="1"/>
+<wire x1="25.42" y1="14.82" x2="24.4" y2="13.8" width="0.3048" layer="1"/>
+<wire x1="24.4" y1="13.8" x2="24.4" y2="13.3" width="0.3048" layer="1"/>
+<wire x1="24.4" y1="13.3" x2="23.7" y2="12.6" width="0.3048" layer="1"/>
+<wire x1="23.7" y1="12.6" x2="22.428425" y2="12.6" width="0.3048" layer="1"/>
+<wire x1="22.428425" y1="12.6" x2="20.4495375" y2="10.6211125" width="0.3048" layer="1"/>
 </signal>
 <signal name="IO7">
@@
 </signal>
 <signal name="IRLED">
-<contactref element="U3" pad="9"/>
 <contactref element="IR" pad="A"/>
-<wire x1="14.944571875" y1="14.015225" x2="13.2" y2="15.759796875" width="0.4064" layer="1"/>
-<wire x1="13.2" y1="15.759796875" x2="13.2" y2="16.4" width="0.4064" layer="1"/>
-<via x="13.2" y="16.4" extent="1-16" drill="0.4318"/>
-<wire x1="13.2" y1="16.4" x2="14" y2="17.2" width="0.4064" layer="16"/>
-<wire x1="14" y1="17.2" x2="33.4" y2="17.2" width="0.4064" layer="16"/>
-<wire x1="33.4" y1="17.2" x2="34.6" y2="16" width="0.4064" layer="16"/>
-<wire x1="34.6" y1="16" x2="35.73" y2="16" width="0.4064" layer="16"/>
+<contactref element="U3" pad="1"/>
+<wire x1="21.015225" y1="10.055425" x2="21.015225" y2="10.115225" width="0.3048" layer="1"/>
+<wire x1="21.015225" y1="10.115225" x2="22.7" y2="11.8" width="0.3048" layer="1"/>
+<wire x1="22.7" y1="11.8" x2="24.2" y2="11.8" width="0.3048" layer="1"/>
+<wire x1="24.2" y1="11.8" x2="25.4" y2="13" width="0.3048" layer="1"/>
+<wire x1="25.4" y1="13" x2="29.9" y2="13" width="0.3048" layer="1"/>
+<wire x1="29.9" y1="13" x2="32.9" y2="16" width="0.3048" layer="1"/>
+<wire x1="32.9" y1="16" x2="35.73" y2="16" width="0.3048" layer="1"/>
 </signal>
 <signal name="WS2812">
